File: VLR-MBHP_MF_NG/MBPH_MF_NGv1.3.1.brd (EAGLE design)
At the start: 140 x 59.8 mm, 51 parts, among them J40 MF_I/O, J41 MF_I/O to more MF_NG

Commit message: div. changes
Parts:
- added U$5: (no value), Frames_VLR:VLRLAB_SMAL
- added U$6: (no value), Frames_VLR:VLRLAB
- moved END+ 11.4 mm to (124.4, 16.9)
- moved END- 11.3 mm to (124.6, 5.00)
Connections:
- net MF_NG-RX_M+: now also J40.6; no longer J40.1
- net MF_NG-RX_M-: now also J40.2; no longer J40.5
- net MF_NG_ENDPOINT_TX+: now also J40.5, J41.6; no longer J40.2, J41.2
- net MF_NG_ENDPOINT_TX-: now also J40.1, J41.2; no longer J40.6, J41.6
Routing:
- net MF_NG-TX+: track 30.2 -> 37.2 mm
- net MF_NG_ENDPOINT_TX+: track 135.4 -> 139.8 mm
- net MF_NG-TX-: track 18.1 -> 20.2 mm
- net MF_NG_ENDPOINT_TX-: track 135.5 -> 137.4 mm, vias 2 -> 1
- net MF_NG-RX_M-: track 24.2 -> 22.7 mm
- net MF_NG-RX_M+: track 11.4 -> 10.0 mm
Other:
- board text added: "(C)Midibox.org, VLRlab.com MF_NG V1.3.1"
