File: VLR-MBHP_MF_NG/MF_NG.sch (EAGLE design)
At the start: 51 parts, among them J40 MF_I/O, J41 MF_I/O to more MF_NG

Commit message: update MF_NGv2.0.1
Parts:
- removed END+, END-: 1, Jumper:SJ
- removed J40: MF_I/O, con-ml:ML6
- removed J41: MF_I/O to more MF_NG, con-ml:ML6
- removed MF_D1: 1N4148, diode:1N4148DO35-7
- removed MF_IC9: 6N138, optocoupler:6N138
- removed MF_R11, MF_R7, MF_R8: 220, resistor:R-EU_0204/7
- removed MF_R5: 4.7k, resistor:R-EU_0204/7
- removed MF_R6: 1k, resistor:R-EU_0204/7
- added J1, J2: (no value), con-ml_Ivan:ML10ML10_TEXTFRONT
- added M-IN, M-OUT: SJ2X4MIDI, Jumper:SJ2X4MIDI
- MF_C21, MF_C23, MF_C7, MF_C8, MF_C9: device capacitor-wima:C5/3 -> rcl:C-EU025-025X050
Connections:
- removed net MF_NG-RX_M+: J40.6, MF_R11.2
- removed net MF_NG-RX_M-: J40.2, MF_D1.A, MF_IC9.C
- removed net MF_NG-TX+: END+.1, J41.1, MF_R8.1
- removed net MF_NG-TX-: END-.2, J41.5, MF_R7.1
- removed net MF_NG_ENDPOINT_TX+: END+.2, J40.5, J41.6
- removed net MF_NG_ENDPOINT_TX-: END-.1, J40.1, J41.2
- removed net N$101: MF_D1.C, MF_IC9.A, MF_R11.1
- removed net N$76: MF_IC9.VB, MF_R5.1
- new net N$10: J2.5, M-OUT.M4
- new net N$11: J1.8, M-IN.I1
- new net N$12: J1.7, M-IN.I2
- new net N$13: J1.10, M-IN.I3
- new net N$14: J1.9, M-IN.I4
- new net N$15: J2.8, M-IN.M1
- new net N$16: J2.7, M-IN.M2
- new net N$17: J2.10, M-IN.M3
- new net N$18: J2.9, M-IN.M4
- new net N$3: J1.4, M-OUT.I1
- new net N$4: J1.3, M-OUT.I2
- new net N$5: J1.6, M-OUT.I3
- new net N$6: J1.5, M-OUT.I4
- new net N$7: J2.4, M-OUT.M1
- new net N$8: J2.3, M-OUT.M2
- new net N$9: J2.6, M-OUT.M3
- net +5V: now also J1.2, J2.2; no longer MF_IC9.VCC, MF_R6.1, MF_R8.2
- net GND: now also J1.1, J2.1; no longer J40.3, J40.4, J41.3, J41.4, MF_IC9.GND, MF_R5.2
- net MIDI_MF_NG-RX: now also M-IN.0; no longer MF_IC9.VO, MF_R6.2
- net MIDI_MF_NG-TX: now also M-OUT.0; no longer MF_R7.2
Other:
- note added: "J1 is the Connectionport to the Core. To get MF alive you need to set two solderpoints. One for the Incoming Data and one for the outgoing Data. Due to the option of chaining 4 Modules its necassary to set the connections on M-IN and M-OUT right. Please visit www.vlrlab.com for support."
