File: VLR-MBHP_CORE_STM32F4Disco/MBHP_CORE_STM32F4v1.1.12.sch (EAGLE design)
At the start: 63 parts, among them M1_D1 1N4148DO35-7, M1_IC1 6N138DIL, M1_J1 CR_MIDI1, M1_R1 220, M1_R2 220, M1_R3 220, M1_R4 4.7k, M1_R5 1k, M2_D1 1N4148DO35-7, M2_IC1 6N138DIL, M2_J1 CR_MIDI1, M2_R1 220, M2_R2 220, M2_R3 220, M2_R4 4.7k, M2_R5 1k

Commit message: Untested
New Layout untested. Prototype in production.
Parts:
- removed CR_J16: 3.3V SPI Devices, con-harting-ml:ML10
- removed CR_R33: 1k, Bourns Resistor Array:4306R
- removed CR_SDCARD: ALPS_SCHA5B200, Micro SD:ALPS_SCHA5B200
- removed M1_D1, M2_D1: 1N4148DO35-7, diode:1N4148DO35-7
- removed M1_IC1, M2_IC1: 6N138DIL, 6N138:6N138DIL
- removed M1_J1, M2_J1: CR_MIDI1, con-harting-ml:ML6
- removed M1_R1, M1_R2, M1_R3, M2_R1, M2_R2, M2_R3: 220, resistor:R-EU_0204/7
- removed M1_R4, M2_R4: 4.7k, resistor:R-EU_0204/7
- removed M1_R5, M2_R5: 1k, resistor:R-EU_0204/7
- removed MIDI1_IN, MIDI1_OUT, MIDI2_IN, MIDI2_OUT: MABP5S, midi:MABP5S
- removed U$2: 3M_SD-RSMT-2-MQ, Memory:3M_SD-RSMT-2-MQ
- added C13, C5, C6: (no value), rcl:C-EU025-025X050
- added C4: 10u, rcl:CPOL-EUE2.5-6
- added CR_J2: 5V, pinhead_Ivan:PINHD-1X2
- added D2: 1N4148DO35-7, diode:1N4148DO35-7
- added D3, D4, D5: 1N4148, diode:1N4148DO35-7
- added IC10, IC4, IC6, IC8: 6N138, 6N138:6N138DIL
- added IC16: 74HC125N, 74xx-eu:74HC125N
- added IC5: 74HC00N, 74xx-eu:74AC00N
- added J12: MIDI1, con-harting-ml:ML6
- added J13: MIDI2, con-harting-ml:ML6
- added J16A: SPI, con-harting-ml:ML10
- added J16B: KISSBOX OEM RTP-MIDI, con-harting-ml:ML10
- added J20: MIDI3, con-harting-ml:ML6
- added J21: MIDI4, con-harting-ml:ML6
- added LED1: RX, led:LED3MM
- added LED2: TX, led:LED3MM
- added R18, R23, R28, R4: 1k, resistor:R-EU_0204/7
- added R19, R24, R29, R35: 4.7k, resistor:R-EU_0204/7
- added R20, R21, R22, R25, R26, R27, R30, R31, R32, R36, R37, R38, R6, R8: 220, resistor:R-EU_0204/7
- added R33: 1k, Bourns Resistor Array:4306R
- added R34: 7R_ARRAY, Bourns Resistor Array:7R_ARRAY
- added R5, R7: 100k, resistor:R-EU_0204/7
- added SD: 3M_SD-RSMT-2-MQ, Memory:3M_SD-RSMT-2-MQ
- C3: value (none) -> 10u; device rcl:C-EU025-025X050 -> rcl:CPOL-EUE2.5-6
- renumbered CR_8B to R8B, CR_C2 to C12, CR_D1 to D1, CR_IC1 to IC1, CR_IC2 to IC2, CR_IC3 to IC7, CR_J10A to J10A, CR_J10B to J10B, CR_J11E to J11E, CR_J15A to J15A, CR_J15B to J15B, CR_J15_S to J15_S, CR_J18 to J18, CR_J19 to J19, CR_J30 to J30, CR_J4A to J4A, CR_J4B to J4B, CR_J5A to J5A, CR_J5B to J5B, CR_J8/9 to J8/9, CR_P1 to P1, CR_P2 to P2, CR_R1 to R1, CR_R12 to R12, CR_R13 to R13, CR_R15 to R15, CR_R2 to R2, CR_R3 to R3, CR_R7A to R7A, CR_R7B to R7B, CR_R8A to R8A, CR_T1 to T1, KLEMME3 to J1B, KLEMME4 to J1A
Connections:
- removed net J_8/9-SI: J8/9.5
- removed net M1_R4: M1_IC1.VB, M1_R4.1
- removed net M1_RX+: M1_J1.5, M1_R3.2, MIDI1_IN.4
- removed net M1_RX+D1: M1_D1.C, M1_IC1.A, M1_R3.1
- removed net M1_RX-: M1_D1.A, M1_IC1.C, M1_J1.1, MIDI1_IN.5
- removed net M1_TX+: M1_J1.6, M1_R2.1, MIDI1_OUT.4
- removed net M1_TX-: M1_J1.2, M1_R1.1, MIDI1_OUT.5
- removed net M2_R4: M2_IC1.VB, M2_R4.1
- removed net M2_RX+: M2_J1.5, M2_R3.2, MIDI2_IN.4
- removed net M2_RX+D1: M2_D1.C, M2_IC1.A, M2_R3.1
- removed net M2_RX-: M2_D1.A, M2_IC1.C, M2_J1.1, MIDI2_IN.5
- removed net M2_TX+: M2_J1.6, M2_R2.1, MIDI2_OUT.4
- removed net M2_TX-: M2_J1.2, M2_R1.1, MIDI2_OUT.5
- new net CR_M1-: D2.A, IC4.C, J12.1
- new net CR_M2+$1: D2.C, IC4.A, R20.1
- new net MF_M+ZULEITUNG: J13.5, R25.2
- new net MF_M+ZULEITUNG1: J20.5, R30.2
- new net MF_M+ZULEITUNG2: J21.5, R36.2
- new net MF_M-ZULEITUNG: D4.A, IC6.C, J13.1
- new net MF_M-ZULEITUNG1: D3.A, IC8.C, J20.1
- new net MF_M-ZULEITUNG2: D5.A, IC10.C, J21.1
- new net N$11: IC4.VB, R19.1
- new net N$13: IC16A.O, IC16B.O
- new net N$19: D4.C, IC6.A, R25.1
- new net N$20: J12.5, R20.2
- new net N$21: C3.-, IC5C.I0, IC5C.I1, R5.1
- new net N$22: C3.+, IC5D.O
- new net N$23: IC5C.O, IC5D.I0, R6.2
- new net N$25: J13.6, R27.1
- new net N$26: J13.2, R26.1
- new net N$27: LED1.C, R6.1
- new net N$28: D3.C, IC8.A, R30.1
- new net N$29: IC8.VB, R29.1
- new net N$30: J20.6, R32.1
- new net N$31: J20.2, R31.1
- new net N$32: D5.C, IC10.A, R36.1
- new net N$33: IC10.VB, R35.1
- new net N$34: J21.6, R38.1
- new net N$35: J21.2, R37.1
- new net N$36: IC5B.I0, IC5B.I1
- new net N$37: C4.-, R7.1
- new net N$39: C4.+, IC5A.O
- new net N$40: IC5A.I1, IC5B.O, R8.2
- new net N$42: LED2.C, R8.1
- new net N$5: R34.2, SD.DATA2
- new net N$6: IC16B.I, J16B.9
- new net N$7: R34.7, SD.DATA1
- new net N$81: J12.2, R21.1
- new net N$99: IC6.VB, R24.1
- new net RTP_IO1: J16B.1
- new net RTP_IO2: J16B.2
- new net RTP_IO3: J16B.5
- new net RTP_IO4: J16B.8
- new net SD_SS: STM32F4DISCOVERY.BOOT0
- net +3V3: now also C13.1, J16A.3, J16A.4, R22.2, R27.2, R32.2, R34.1, R38.2, SD.VDD; no longer C2.1, CR_J16.3, CR_J16.4, CR_SDCARD.VDD, M1_R2.2, M2_R2.2, STM32F4DISCOVERY.VDD, STM32F4DISCOVERY.VDD1, STM32F4DISCOVERY.VDD3, STM32F4DISCOVERY.VDD4, U$2.VDD
- net +5V: now also C5.2, C6.2, CR_J2.2, IC10.VCC, IC16P.VCC, IC4.VCC, IC5P.VCC, IC6.VCC, IC8.VCC, J16B.3, J4B.10, LED1.A, LED2.A, R18.1, R23.1, R28.1, R4.1; no longer J4B.4, M1_IC1.VCC, M1_R5.1, M2_IC1.VCC, M2_R5.1
- net DIN_SI: now also J8/9.5
- net GND: now also C13.2, C5.1, C6.1, CR_J2.1, IC10.GND, IC16P.GND, IC4.GND, IC5P.GND, IC6.GND, IC8.GND, J12.4, J13.4, J16A.1, J16A.2, J16B.4, J20.4, J21.4, J4A.1, J4A.2, J4A.3, J4A.5, J4A.7, J4A.9, J4B.1, J4B.2, J4B.3, J4B.4, J4B.5, J4B.7, J4B.9, R19.2, R24.2, R29.2, R35.2, R5.2, R7.2, SD.GND1,2, SD.VSS; no longer C3.2, CR_J16.1, CR_J16.2, CR_SDCARD.GND, CR_SDCARD.VSS, J4B.10, M1_IC1.GND, M1_J1.4, M1_R4.2, M2_IC1.GND, M2_J1.4, M2_R4.2, MIDI1_IN.PE, MIDI1_OUT.PE, MIDI2_IN.PE, MIDI2_OUT.PE, U$2.GND1,2, U$2.VSS
- net LCD_E1: now also R33.2; no longer CR_R33.6
- net LCD_E2: now also R33.5; no longer CR_R33.3
- net LCD_RS: now also R33.4; no longer CR_R33.5
- net LCD_RW: now also R33.6; no longer CR_R33.4
- net LCD_VOLTAGE_OPTION: now also C2.1, R33.1; no longer C3.1, CR_R33.1
- net MI1: now also IC4.VO, IC5D.I1, R18.2; no longer M1_IC1.VO, M1_R5.2
- net MI2: now also IC6.VO, R23.2; no longer M2_IC1.VO, M2_R5.2
- net MI3: now also IC8.VO, R28.2
- net MI4: now also IC10.VO, R4.2
- net MO1: now also IC5A.I0, R21.2; no longer M1_R1.2
- net MO2: now also R26.2; no longer M2_R1.2
- net MO3: now also R31.2
- net MO4: now also R37.2
- net N$16: now also J12.6, R22.1; no longer M2_J1.3
- net N$24: now also J12.3; no longer M1_J1.3
- net SPI_RC1: now also IC16A.OE, J16A.10, R34.3, SD.CD/DATA3; no longer CR_J16.10, CR_SDCARD.CD/DATA3, U$2.CD/DATA3
- net SPI_RC2: now also IC16B.OE, J16A.9, J16B.6; no longer CR_J16.9
- net SPI_SC: now also J16A.7, J16A.8, J16B.7, R34.5, SD.CLK; no longer CR_J16.7, CR_J16.8, CR_SDCARD.CLK, U$2.CLK
- net SPI_SI: now also IC16A.I, J16A.5, R34.6, SD.DATA0; no longer CR_J16.5, CR_SDCARD.DATA0, U$2.DATA0
- net SPI_SO: now also J16A.6, J16B.10, R34.4, SD.CMD; no longer CR_J16.6, CR_SDCARD.CMD, U$2.CMD
Other:
- moved on the sheet: C2
