File: VLR-MBHP_CORE_STM32F4Disco/MBHP_CORE_STM32F4.brd (EAGLE design)
At the start: 120 x 140 mm, 91 parts, among them IC1 74HC541, IC10 6N138, IC16 74HC125N, IC2 74HC595, IC4 6N138, IC5 74HC00N, IC6 6N138, IC7 LF33, IC8 6N138, J10A DIGITAL, J10B DIGITAL, J11E MOSI, J12 MIDI1, J13 MIDI2, J15A Disp1, J15B Disp2, J15_S LCD Volt. Opt., J16A SPI, J16B KISSBOX OEM RTP-MIDI, J18 CAN, J19 AOUT/SPI, J1A PT-1.5/3, J1B PT-1.5/3, J20 MIDI3, J21 MIDI4, J30 DISP-EXT, J4A IIC1, J4B IIC2, J5A ANALOG, J5B ANALOG, J8/9 DIN/DOUT, P1 10k, P2 10k, T1 BC337

Commit message: update to STMF4v.2.2.1
Parts:
- removed R15: 1k, resistor:0204/7
- added R11: 1k, resistor:0204/7
- added U$1, U$2: KEYSTONE_SCREW_TERMINAL, holes_Ivan:KEYSTONE_SCREW_TERMINAL
- C12: value 100 -> 100uF
- C13, C5, C6: value (none) -> 100nF
- J10A: value DIGITAL -> DIGITAL A
- J10B: value DIGITAL -> DIGITAL B
- R34: value 7R_ARRAY -> 10k
- moved J18 111.0 mm to (44.3, 111.3)
- moved D1 60.5 mm to (43.0, 104.7), turned to 90 degrees
- moved U$6 42.9 mm to (4.07, 61.9)
- moved C2 11.1 mm to (93.8, 65.2)
- moved R33 11.0 mm to (82.6, 65.5)
- moved IC2 10.9 mm to (86.2, 57.5)
- moved U$7 8.90 mm to (4.29, 120.4), turned to 0 degrees
- moved R7A 2.92 mm to (84.1, 30.9)
- moved R8A 2.90 mm to (86.4, 30.9)
- moved R8 0.62 mm to (6.62, 21.3)
- moved R3 0.30 mm to (80.0, 121.3)
- moved R1 0.20 mm to (77.7, 121.4)
- moved R2 0.20 mm to (75.4, 121.4)
Connections:
- net +3V3: no longer R22.2, R27.2, R32.2, R38.2
- net +5V: now also R11.2, R22.2, R27.2, R32.2, R38.2; no longer R15.2
- net CAN_RX: now also R11.1; no longer R15.1
- net GND: now also SD.6, U$1.P$1, U$1.P$2, U$1.P$3, U$1.P$4, U$2.P$1, U$2.P$2, U$2.P$3, U$2.P$4
Routing:
- net CAN_RX: track 79.2 -> 230.6 mm
- net +3V3: track 385.3 -> 282.8 mm, vias 2 -> 1
- net CAN_TX: track 10.8 -> 87.6 mm, vias 0 -> 1
- net +5V: track 487.5 -> 537.7 mm, vias 1 -> 2
- net RC-O-: track 46.6 -> 30.7 mm
- net LCD_SER_SCLK: track 65.6 -> 79.0 mm
- net LCD_VOLTAGE_OPTION: track 154.2 -> 141.6 mm, vias 2 -> 1
- net N$2: track 29.2 -> 41.6 mm
- net N$1: track 32.3 -> 44.3 mm
- net N$4: track 33.1 -> 44.5 mm
- net LCD_D7: track 94.4 -> 105.5 mm, vias 1 -> 2
- net LCD_RW: track 181.5 -> 191.5 mm, vias 2 -> 3
- net RC-I-: track 43.8 -> 33.8 mm
- net SC-: track 49.5 -> 39.7 mm
- net N$8: track 38.5 -> 47.3 mm
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Other:
- board text added: "1"
- board text added: "3.3V"
- board text added: "ANALOG"
- board text added: "AOUT / SPI"
- board text added: "C12"
- board text added: "C13"
- board text added: "CS"
- board text added: "DI"
- board text added: "DIGITAL A"
- board text added: "DIGITAL B"
- board text added: "DIN/DOUT"
- board text added: "DO"
- board text added: "IN"
- board text added: "M+"
- board text added: "M-"
- board text added: "MIDI 1 TEST"
- board text added: "MIDI1"
- board text added: "MIDI2"
- board text added: "MIDI3"
- board text added: "MIDI4"
- board text added: "Midibox Core STM32F407 PCB (C) T.Klose / I.Hörler / B.Bouchez Version 2.2.1 / RTP Ready"
- board text added: "SCLK"
- board text added: "SPI"
- board text removed: "(C) Midibox.org, VLRlab.com Fadercore 2.1.1"
- board text removed: "AOUT/SPI"
- board text removed: "DIGITAL"
- board text removed: "DISP1"
- board text removed: "DISP2"
- board text removed: "H"
- board text removed: "IC04"
- board text removed: "IC06"
- board text removed: "IC08"
- board text removed: "IC1"
- board text removed: "IC10"
- board text removed: "IC2"
- board text removed: "IN+"
- board text removed: "IN-"
- board text removed: "J10A"
- board text removed: "J11E"
- board text removed: "J12"
- board text removed: "J13"
- board text removed: "J16B"
- board text removed: "J19"
- board text removed: "J20"
- board text removed: "J21"
- board text removed: "MIDI 4 TEST"
