File: VLR-MBHP_CORE_STM32F4Disco/MBHP_CORE_STM32F4.sch (EAGLE design)
At the start: 89 parts, among them IC1 74HC541, IC10 6N138, IC16 74HC125N, IC2 74HC595, IC4 6N138, IC5 74HC00N, IC6 6N138, IC7 LF33, IC8 6N138, J10A DIGITAL, J10B DIGITAL, J11E MOSI, J12 MIDI1, J13 MIDI2, J15A Disp1, J15B Disp2, J15_S LCD Volt. Opt., J16A SPI, J16B KISSBOX OEM RTP-MIDI, J18 CAN, J19 AOUT/SPI, J1A PT-1.5/3, J1B PT-1.5/3, J20 MIDI3, J21 MIDI4, J30 DISP-EXT, J4A IIC1, J4B IIC2, J5A ANALOG, J5B ANALOG, J8/9 DIN/DOUT, P1 10k, P2 10k, T1 BC337

Commit message: update to STMF4v.2.2.1
Parts:
- added U$1, U$2: KEYSTONE_SCREW_TERMINAL, holes_Ivan:KEYSTONE_SCREW_TERMINAL
- C12: value 100 -> 100uF
- C13, C5, C6: value (none) -> 100nF
- J10A: value DIGITAL -> DIGITAL A
- J10B: value DIGITAL -> DIGITAL B
- R34: value 7R_ARRAY -> 10k
- renumbered R15 to R11
Connections:
- net +3V3: no longer R22.2, R27.2, R32.2, R38.2
- net +5V: now also R22.2, R27.2, R32.2, R38.2
- net GND: now also SD.GND, U$1G$1.GND, U$1G$2.GND, U$1G$3.GND, U$1G$4.GND, U$2G$1.GND, U$2G$2.GND, U$2G$3.GND, U$2G$4.GND
