File: VLR-8x16LEDmeter/LEDmatrixboard/LEDmatrixboard.brd (EAGLE design)
At the start: 59.8 x 140 mm, 23 parts, among them IC1 74HC595, IC2 74HC595, IC3 74HC595

Commit message: update LEDMatrixboardV2.2.1
Parts:
- removed R1-8: 220, Bourns Resistor Array:SOIC16W
- added IC5: ULN2803, 595-541-165-uln2803:SO18W
- moved IC1 3.14 mm to (11.3, 28.0), turned to 270 degrees
- moved C1 1.17 mm to (18.8, 22.0)
Connections:
- net +5V: now also IC5.10
- net GND: now also IC5.9
- net N$1: now also IC1.7, IC5.8; no longer IC1.15, R1-8.16
- net N$34: now also IC1.6, IC5.7; no longer IC1.1, R1-8.15
- net N$35: now also IC1.5, IC5.6; no longer IC1.2, R1-8.14
- net N$36: now also IC1.4, IC5.5; no longer IC1.3, R1-8.13
- net N$37: now also IC1.3, IC5.4; no longer IC1.4, R1-8.12
- net N$38: now also IC1.2, IC5.3; no longer IC1.5, R1-8.11
- net N$39: now also IC1.1, IC5.2; no longer IC1.6, R1-8.10
- net N$40: now also IC1.15, IC5.1; no longer IC1.7, R1-8.9
- net N$41: now also IC5.11; no longer R1-8.1
- net N$42: now also IC5.12; no longer R1-8.2
- net N$43: now also IC5.13; no longer R1-8.3
- net N$44: now also IC5.14; no longer R1-8.4
- net N$45: now also IC5.15; no longer R1-8.5
- net N$46: now also IC5.16; no longer R1-8.6
- net N$47: now also IC5.17; no longer R1-8.7
- net N$48: now also IC5.18; no longer R1-8.8
Routing:
- net N$40: track 3.89 -> 32.4 mm
- net +5V: track 210.0 -> 194.3 mm, vias 2 -> 4
- net N$72: track 164.7 -> 177.3 mm
- net N$34: track 3.89 -> 15.0 mm
- net N$35: track 3.89 -> 13.0 mm
- net N$36: track 3.89 -> 11.0 mm
- net N$1: track 10.4 -> 17.1 mm
- net N$66: track 35.2 -> 29.2 mm
- net N$49: track 21.7 -> 16.5 mm, vias 0 -> 2
- net N$37: track 3.89 -> 9.05 mm
- net N$38: track 3.89 -> 7.21 mm
- net N$71: track 200.0 -> 202.9 mm, vias 2 -> 3
- net N$45: track 48.1 -> 45.2 mm
- net N$46: track 58.2 -> 55.3 mm
- net N$48: track 78.2 -> 75.3 mm
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Other:
- board text added: "(C)VLRlab.com Matrixboard V2.2.1"
- board text added: "GND"
- board text added: "J1"
- board text added: "J2"
- board text added: "RC-I"
- board text added: "RC-O"
- board text added: "ROW1"
- board text added: "ROW10"
- board text added: "ROW11"
- board text added: "ROW12"
- board text added: "ROW13"
- board text added: "ROW14"
- board text added: "ROW15"
- board text added: "ROW16"
- board text added: "ROW2"
- board text added: "ROW3"
- board text added: "ROW4"
- board text added: "ROW5"
- board text added: "ROW6"
- board text added: "ROW7"
- board text added: "ROW8"
- board text added: "ROW9"
- board text added: "SC"
- board text added: "SEL1"
- board text added: "SEL2"
- board text added: "SEL3"
- board text added: "SEL4"
- board text added: "SEL5"
- board text added: "SEL6"
- board text added: "SEL7"
- board text added: "SEL8"
- board text added: "SI"
- board text added: "SO"
- board text removed: "(C)VLRlab.com Matrixboard V1.2.4"
