File: VLR-MBHP_DOUT/DOUT.brd (EAGLE design)
At the start: 59.8 x 140 mm, 28 parts, among them IC2 74HC595, IC3 74HC595, IC4 74HC595

Commit message: comliant changes v1.3
Parts:
- added U$2, U$3: (no value), Beschriftungen:DOUT
- added U$4, U$5: (no value), Frames_VLR:VLRLAB
Changed lines of the file:
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@@
 <?xml version="1.0" encoding="utf-8"?>
 <!DOCTYPE eagle SYSTEM "eagle.dtd">
-<eagle version="7.1.0">
+<eagle version="7.2.0">
 <drawing>
 <settings>
@@
 <setting verticaltext="up"/>
 </settings>
-<grid distance="10" unitdist="mil" unit="mil" style="lines" multiple="1" display="yes" altdistance="1" altunitdist="mil" altunit="mil"/>
+<grid distance="0.05" unitdist="inch" unit="inch" style="lines" multiple="1" display="no" altdistance="0.025" altunitdist="inch" altunit="inch"/>
 <layers>
 <layer number="1" name="Top" color="4" fill="1" visible="yes" active="yes"/>
@@
 <element name="SJ7" library="Jumper" package="SJ" value="" x="37.592" y="62.738" rot="R180"/>
 <element name="SJ8" library="Jumper" package="SJ" value="" x="37.592" y="35.306" rot="R180"/>
+<element name="U$2" library="Beschriftungen" package="DOUT" value="" x="40.64" y="133.35"/>
+<element name="U$3" library="Beschriftungen" package="DOUT" value="" x="52.07" y="133.35" rot="MR0"/>
+<element name="U$4" library="Frames_VLR" package="VLRLAB" value="" x="41.91" y="3.81"/>
+<element name="U$5" library="Frames_VLR" package="VLRLAB" value="" x="53.34" y="3.81" rot="MR0"/>
 </elements>
 <signals>
@@
 </board>
 </drawing>
+<compatibility>
+<note version="6.3" minversion="6.2.2" severity="warning">
+Since Version 6.2.2 text objects can contain more than one line,
+which will not be processed correctly with this version.
+</note>
+</compatibility>
 </eagle>
